File: Controller_board.kicad_pcb (KiCad board)
At the start: 4 copper layers, 100 x 65 mm, 88 parts, among them J1 USB_B_Micro, J2 OLED_CONN, J3 SWD + UART, J4 SMA, Q1 BXT520P02M, Q2 DMP2045U, Q3 BC847-QR, SW1 SW_SPDT, SW2 Rotary Encoder, SW3 SW_Push, SW4 SW_Push, U1 LD1117S33CTR, U2 MIC2288, U3 USBLC6-2SC6, U4 STM32F401RBT6, U5 MPU-6050, U6 nRF24L01P, U7 M24C02-FMN, U8 COM-09032, U9 COM-09032, Y1 16 MHz, Y2 16 MHz

Commit message: Added Gerbers
Parts:
- removed TP1: Test 5V, TestPoint:TestPoint_Pad_D1.0mm
- added TP5: NRF_TestPoint_CSN, TestPoint:TestPoint_Pad_D1.0mm, B.Cu at (115.7, 99.1)
- added TP6: NRF_TestPoint_CE, TestPoint:TestPoint_Pad_D1.0mm, B.Cu at (113.3, 99.1)
- added TP7: NRF_TestPoint_IRQ, TestPoint:TestPoint_Pad_D1.0mm, B.Cu at (118.0, 99.1)
- C14, C15, C22, C23, C24, C25, C26, C27, C29: footprint Capacitor_SMD:C_0402_1005Metric -> Capacitor_SMD:C_0603_1608Metric
- J4: footprint digikey-footprints:RF_SMA_BoardEdge_142-0701-801 -> Connector_Coaxial:SMA_Molex_73251-2120_EdgeMount_Horizontal
- JP1, SW1: moved to B.Cu
- L3, L4, L5: footprint Inductor_SMD:L_0402_1005Metric -> Inductor_SMD:L_0603_1608Metric
- moved R6 4.75 mm to (128.5, 107.4), turned to 90 degrees
- moved L4 2.84 mm to (115.1, 94.1)
- moved U6 2.57 mm to (115.0, 97.7)
- moved C5 2.50 mm to (107.7, 103.8), turned to 180 degrees
- moved R13 2.34 mm to (110.2, 96.3)
- moved C18 2.34 mm to (110.2, 94.4)
- moved C24 2.25 mm to (122.5, 99.8)
- moved L3 2.04 mm to (114.3, 91.8)
- moved C19 2.02 mm to (119.6, 99.9)
- moved R12 2.02 mm to (119.6, 95.9)
- moved Y2 2.02 mm to (122.5, 96.8)
- moved J4 2.01 mm to (115.0, 82.4), turned to 90 degrees
- moved D4 1.97 mm to (126.7, 107.4), turned to -90 degrees
- moved R3 1.96 mm to (95.8, 106.7)
- moved C26 1.83 mm to (118.9, 88.8)
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Connections:
- R3 pad 1: +5V -> +3.3V
Routing:
- net -BATT: track 76.5 -> 90.0 mm, vias 98 -> 91
- net +3.3V: track 62.5 -> 69.3 mm
- net +5V: track 10.2 -> 4.94 mm
- net NRF_VDD_PA: track 5.00 -> 8.40 mm
- net LATCH_POWERUP: track 4.60 -> 7.29 mm, vias 0 -> 1
- net NRF_MOSI: track 10.4 -> 8.07 mm
- net +BATT: track 13.7 -> 16.0 mm
- net NRF_MISO: track 8.85 -> 6.88 mm
- net NRF_ANT1: track 3.12 -> 5.04 mm
- net NRF_SCK: track 11.0 -> 9.31 mm
- net BATTERY_ADC: track 49.6 -> 48.1 mm
- net Net-(U4-VCAP1): track 3.69 -> 2.59 mm
- net Net-(D4-K): track 6.30 -> 7.23 mm
- net Net-(C22-Pad2): track 5.25 -> 6.12 mm
- net NRF_CSN: track 7.51 -> 8.35 mm, vias 0 -> 1
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Other:
- board text added: "3.3V"
- board text added: "CE"
- board text added: "CSN"
- board text added: "DISP"
- board text added: "DWN"
- board text added: "Designed by M.Klebokowski"
- board text added: "ENC"
- board text added: "IRQ"
- board text added: "Klecontroller"
- board text added: "L-ANALOG"
- board text added: "R-ANALOG"
- board text added: "RF 2.4GHz Klebot Controller rev 1.0 - 10/23"
- board text added: "UP"
- board text added: "USB"
- board text removed: "+3.3V"
- board text removed: "+5V"
- board text removed: "BATT"
- board text removed: "OLED"
- board text removed: "nRF Controller"
- board text removed: "nRF Controller rev 1.0 - 07/23"
