File: Controller_board.kicad_sch (KiCad schematic)
At the start: 0 parts

Commit message: finalising layout
Parts:
- added BT1: Battery, TerminalBlock_Phoenix:TerminalBlock_Phoenix_PT-1,5-2-3.5-H_1x02_P3.50mm_Horizontal, symbol Device:Battery
- added C1, C16: 4u7, Capacitor_SMD:C_0603_1608Metric, symbol Device:C_Small
- added C10, C9: 100nF, Capacitor_SMD:C_0603_1608Metric, symbol Device:C_Small
- added C11: 10uF, Capacitor_SMD:C_0603_1608Metric, symbol Device:C_Small
- added C12: 1u, Capacitor_SMD:C_0603_1608Metric, symbol Device:C_Small
- added C13: 10n, Capacitor_SMD:C_0603_1608Metric, symbol Device:C_Small
- added C14, C15: 10p, Capacitor_SMD:C_0402_1005Metric, symbol Device:C_Small
- added C2, C3, C4, C5, C6: 100n, Capacitor_SMD:C_0603_1608Metric, symbol Device:C_Small
- added C7: 4u7 6.3V, Capacitor_SMD:C_0603_1608Metric, symbol Device:C_Small
- added C8: 22uF 6.3V, Capacitor_SMD:C_0805_2012Metric, symbol Device:C_Small
- added D1: BAT54C, Package_TO_SOT_SMD:SOT-23, symbol Diode:BAT54C
- added D2, D5: 40V 1A, Diode_SMD:D_SOD-123, symbol Device:D_Schottky_Small
- added D3: LED RED, LED_SMD:LED_0603_1608Metric, symbol Device:LED_Small
- added D4: LED BLUE, LED_SMD:LED_0603_1608Metric, symbol Device:LED
- added FB1: 120R, Inductor_SMD:L_0603_1608Metric, symbol Device:FerriteBead_Small
- added J1: USB_B_Micro, Connector_USB:USB_Micro-B_Amphenol_10103594-0001LF_Horizontal, symbol Connector:USB_B_Micro
- added J2: OLED_CONN, DF3A-4P-2DSA:SHDR4W55P0X200_1X4_1000X500X530P, symbol Connector_Generic:Conn_01x04
- added J3: SWD + UART, Connector_PinHeader_2.00mm:PinHeader_2x05_P2.00mm_Vertical, symbol Connector_Generic:Conn_02x05_Odd_Even
- added JP1: Powerup Mode, Jumper:SolderJumper-3_P1.3mm_Open_RoundedPad1.0x1.5mm, symbol Jumper:SolderJumper_3_Open
- added L1: 4.7uH 650mA, Inductor_SMD:L_1812_4532Metric, symbol Device:L_Small
- added Q1: BXT520P02M, Package_TO_SOT_SMD:SOT-23, symbol SparkFun-DiscreteSemi:MOSFET_PCH-IRLML2244
- added Q2: DMP2045U, Package_TO_SOT_SMD:SOT-23, symbol SparkFun-DiscreteSemi:MOSFET_PCH-IRLML2244
- added Q3: BC847-QR, Package_TO_SOT_SMD:SOT-23, symbol Simulation_SPICE:NPN
- added R1: 5k62, Resistor_SMD:R_0603_1608Metric, symbol Device:R_Small
- added R10, R7, R8, R9: 2k2, Resistor_SMD:R_0603_1608Metric, symbol Device:R_Small
- added R11: 10k, Resistor_SMD:R_0603_1608Metric, symbol Device:R
- added R16, R17, R18: 100k, Resistor_SMD:R_0603_1608Metric, symbol Device:R_Small
- added R2, R5: 100k, Resistor_SMD:R_0603_1608Metric, symbol Device:R
- added R3: 330R, Resistor_SMD:R_0603_1608Metric, symbol Device:R_Small
- added R4: 1k87, Resistor_SMD:R_0603_1608Metric, symbol Device:R_Small
- added R6: ?, Resistor_SMD:R_0603_1608Metric, symbol Device:R
- added SW1: SW_SPDT, Jumper:SolderJumper-3_P1.3mm_Open_RoundedPad1.0x1.5mm, symbol Switch:SW_SPDT
- added TP1: Test 5V, TestPoint:TestPoint_Pad_D1.0mm, symbol Connector:TestPoint
- added U1: LD1117S33CTR, digikey-footprints:SOT-223, symbol dk_PMIC-Voltage-Regulators-Linear:LD1117S33CTR
- added U2: MIC2288, Package_TO_SOT_SMD:TSOT-23-5, symbol Zalfon-kicad-lib:MIC2288
- added U3: USBLC6-2SC6, Package_TO_SOT_SMD:SOT-23-6, symbol Power_Protection:USBLC6-2SC6
- added U4: STM32F401RBT6, Package_QFP:LQFP-64_10x10mm_P0.5mm, symbol MCU_ST_STM32F4:STM32F401RBTx
- added Y1: 16 MHz, Crystal:Crystal_SMD_3225-4Pin_3.2x2.5mm, symbol Device:Crystal_GND24_Small
Connections:
- new net: D4.1 (K), U4.28 (PB2)
- new net: D4.2 (A), R6.1
- new net: C16.1, U4.30 (VCAP1)
- new net: C14.1, U4.5 (PH0), Y1.1
- new net: C15.1, U4.6 (PH1), Y1.3
- new net: R11.2, SW1.2 (B)
- new net: D3.2 (A), R3.2
- new net: C7.1, L1.1, Q1.2 (S), U2.5 (VIN)
- new net: D2.2 (A), L1.2, U2.1 (SW)
- new net: D1.2, Q2.1 (G), Q3.1 (C), R17.2
- new net: Q3.2 (B), R18.1
- new net: C12.1, C13.1, FB1.2, U4.13 (VREF+)
- new net: R1.2, R4.1, U2.3 (FB)
- new net +3.3V: C1.1, C10.1, C11.1, C2.1, C3.1, C4.1, C5.1, C6.1, FB1.1, J2.3 (Pin_3), J3.1 (Pin_1), R10.1, R6.2, R7.1, R8.1, R9.1, SW1.1 (A), U1.2 (VOUT), U1.4 (VOUT), U4.1 (VBAT), U4.19 (VDD), U4.32 (VDD), U4.48 (VDD), U4.64 (VDD)
- new net +5V: C8.1, C9.1, D2.1 (K), D5.1 (K), R1.1, R3.1, TP1.1, U1.3 (VIN)
- new net +BATT: BT1.1 (+), JP1.1 (A), Q1.3 (D), Q2.2 (S), R16.1, R17.1, R2.2
- new net -BATT: BT1.2 (-), C1.2, C10.2, C11.2, C12.2, C13.2, C14.2, C15.2, C16.2, C2.2, C3.2, C4.2, C5.2, C6.2, C7.2, C8.2, C9.2, D3.1 (K), J1.5 (GND), J2.4 (Pin_4), J3.3 (Pin_3), J3.5 (Pin_5), J3.9 (Pin_9), Q1.1 (G), Q3.3 (E), R4.2, R5.1, SW1.3 (C), U1.1 (GND), U2.2 (GND), U3.2 (GND), U4.12 (VSSA), U4.18 (VSS), U4.31 (VSS), U4.47 (VSS), U4.63 (VSS), Y1.2, Y1.4
- new net BATTERY_ADC: R2.1, R5.2, U4.25 (PC5)
- new net BOOT0: R11.1, U4.60 (BOOT0)
- new net BUTTON_DOWN: D1.3
- new net BUTTON_UP: U4.51 (PC10)
- new net EN: JP1.2 (C), U2.4 (EN)
- new net ENC_A: U4.22 (PA6)
- new net ENC_B: U4.23 (PA7)
- new net ENC_BUTTON: U4.21 (PA5)
- new net I2C_SCL: R9.2, U4.61 (PB8)
- new net I2C_SDA: R10.2, U4.62 (PB9)
- new net JOY1_ADC_X: U4.10 (PC2)
- new net JOY1_ADC_Y: U4.9 (PC1)
- new net JOY1_BUTTON: U4.8 (PC0)
- new net JOY2_ADC_X: U4.16 (PA2)
- new net JOY2_ADC_Y: U4.15 (PA1)
- new net JOY2_BUTTON: U4.14 (PA0)
- new net KEEP_ALIVE: R18.2, U4.57 (PB5)
- new net LATCH_POWERUP: JP1.3 (B), Q2.3 (D)
- new net MPU-6050_IRQ: U4.2 (PC13)
- new net NRF_CE: U4.38 (PC7)
- new net NRF_CSN: U4.37 (PC6)
- new net NRF_IRQ: U4.33 (PB12)
- new net NRF_MISO: U4.35 (PB14)
- new net NRF_MOSI: U4.36 (PB15)
- new net NRF_SCK: U4.34 (PB13)
- new net NRST: J3.10 (Pin_10), U4.7 (NRST)
- new net OLED_SCL: J2.2 (Pin_2), R7.2, U4.41 (PA8)
- new net OLED_SDA: J2.1 (Pin_1), R8.2, U4.40 (PC9)
- new net Power_Btn: D1.1, R16.2, U4.54 (PD2)
- new net SWCLK: J3.4 (Pin_4), U4.49 (PA14)
- new net SWDIO: J3.2 (Pin_2), U4.46 (PA13)
- new net SWO: J3.6 (Pin_6), U4.55 (PB3)
- new net USB_CONN_D+: J1.3 (D+), U3.3 (I/O2)
- new net USB_CONN_D-: J1.2 (D-), U3.1 (I/O1)
- new net USB_D+: U3.4 (I/O2), U4.45 (PA12)
- new net USB_D-: U3.6 (I/O1), U4.44 (PA11)
- new net V_USB: D5.2 (A), J1.1 (VBUS), U3.5 (VBUS)
- no-connect marks 0 -> 22
Other:
- removed sheet 18650 Power Supply
- added sheet Peripherals (peripherals.kicad_sch)
- note added: "0,24V Drop"
- note added: "3.3V Regulator"
- note added: "5V Boost Converter (500 mA)"
- note added: "Analog side filtering. Place it between VREF+ and VSSA !"
- note added: "Battery"
- note added: "Battery voltage measurement"
- note added: "Boot switch"
- note added: "Cload = 2 * (CL - Cstray[6])"
- note added: "Connectors"
- note added: "Find 5V tolerant MCU pin!"
- note added: "I2C Pull-up's"
- note added: "Place them close to uC!"
- note added: "Vgs < -2.2V"
- note added: "uC Decoupling"
- title: (none) -> MCU & Power Supply

Commit message: Added Gerbers
Parts:
- removed TP1: Test 5V, TestPoint:TestPoint_Pad_D1.0mm, symbol Connector:TestPoint
- C14, C15: footprint Capacitor_SMD:C_0402_1005Metric -> Capacitor_SMD:C_0603_1608Metric
Connections:
- net +3.3V: now also R3.1
- net +5V: no longer R3.1
Other:
- moved on the sheet: C10, C11, C9, U1
