File: peripherals.kicad_sch (KiCad schematic)
At the start: 36 parts, among them J4 SMA, SW2 Rotary Encoder, SW3 SW_Push, SW4 SW_Push, U5 MPU-6050, U6 nRF24L01P, U7 M24C02-FMN, U8 COM-09032, U9 COM-09032, Y3 16 MHz

Commit message: Added Gerbers
Parts:
- added TP1: NRF_TestPoint_CSN, TestPoint:TestPoint_Pad_D1.0mm, symbol Connector:TestPoint_Small
- added TP1: NRF_TestPoint_IRQ, TestPoint:TestPoint_Pad_D1.0mm, symbol Connector:TestPoint_Small
- added TP1: NRF_TestPoint_CE, TestPoint:TestPoint_Pad_D1.0mm, symbol Connector:TestPoint_Small
- C14: footprint Capacitor_SMD:C_0402_1005Metric -> Capacitor_SMD:C_0603_1608Metric
- J4: footprint digikey-footprints:RF_SMA_BoardEdge_142-0701-801 -> Connector_Coaxial:SMA_Molex_73251-2120_EdgeMount_Horizontal
- L3, L4, L5: footprint Inductor_SMD:L_0402_1005Metric -> Inductor_SMD:L_0603_1608Metric
Connections:
- net NRF_CE: now also TP1.1
- net NRF_CSN: now also TP1.1
- net NRF_IRQ: now also TP1.1
Changed lines of the file:
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@@
+    )
+  )
+  (global_label "NRF_CSN" (shape input) (at 149.86 170.434 180) (fields_autoplaced)
+    (effects (font (size 1.27 1.27)) (justify right))
+    (property "Intersheetrefs" "${INTERSHEET_REFS}" (at 138.4875 170.434 0)
+      (effects (font (size 1.27 1.27)) (justify right) hide)
     )
   )
@@
     )
   )
+  (global_label "NRF_IRQ" (shape input) (at 149.86 181.61 180) (fields_autoplaced)
+    (effects (font (size 1.27 1.27)) (justify right))
+    (property "Intersheetrefs" "${INTERSHEET_REFS}" (at 139.0922 181.61 0)
+      (effects (font (size 1.27 1.27)) (justify right) hide)
+    )
+  )
   (global_label "NRF_SCK" (shape input) (at 41.3004 51.9176 180) (fields_autoplaced)
     (effects (font (size 1.27 1.27)) (justify right))
@@
     (effects (font (size 1.27 1.27)) (justify right))
     (property "Intersheetrefs" "${INTERSHEET_REFS}" (at 31.3189 59.5376 0)
+      (effects (font (size 1.27 1.27)) (justify right) hide)
+    )
+  )
+  (global_label "NRF_CE" (shape input) (at 149.86 175.768 180) (fields_autoplaced)
+    (effects (font (size 1.27 1.27)) (justify right))
+    (property "Intersheetrefs" "${INTERSHEET_REFS}" (at 139.8785 175.768 0)
       (effects (font (size 1.27 1.27)) (justify right) hide)
     )
@@
       (effects (font (size 1.27 1.27)) (justify left))
     )
-    (property "Footprint" "Capacitor_SMD:C_0402_1005Metric" (at 125.0696 57.3278 0)
+    (property "Footprint" "Capacitor_SMD:C_0603_1608Metric" (at 125.0696 57.3278 0)
       (effects (font (size 1.27 1.27)) hide)
     )
@@
       (effects (font (size 1.27 1.27)) (justify left))
     )
-    (property "Footprint" "Capacitor_SMD:C_0402_1005Metric" (at 117.4496 57.3278 0)
+    (property "Footprint" "Capacitor_SMD:C_0603_1608Metric" (at 117.4496 57.3278 0)
       (effects (font (size 1.27 1.27)) hide)
     )
@@
     )
   )
+  (symbol (lib_id "Connector:TestPoint_Small") (at 149.86 170.434 0) (unit 1)
+    (in_bom yes) (on_board yes) (dnp no)
+    (property "Reference" "TP1" (at 152.146 169.799 0)
+      (effects (font (size 1.27 1.27)) (justify left))
+    )
+    (property "Value" "NRF_TestPoint_CSN" (at 152.146 172.339 0)
+      (effects (font (size 1.27 1.27)) (justify left))
+    )
+    (property "Footprint" "TestPoint:TestPoint_Pad_D1.0mm" (at 154.94 170.434 0)
+      (effects (font (size 1.27 1.27)) hide)
+    )
+    (property "Datasheet" "~" (at 154.94 170.434 0)
+      (effects (font (size 1.27 1.27)) hide)
+    )
+    (pin "1")
+    (instances
+      (project "Controller_board"
+        (path "/79650e32-6fba-4eaa-902b-d1154ea8c394"
+          (reference "TP1") (unit 1)
+        )
+        (path "/79650e32-6fba-4eaa-902b-d1154ea8c394/7d15cb0c-3f4d-419a-9225-6f102e9a9922"
+          (reference "TP5") (unit 1)
+        )
+      )
+    )
+  )
   (symbol (lib_id "power:GND") (at 125.0696 59.8678 0) (unit 1)
     (in_bom yes) (on_board yes) (dnp no)
@@
         (path "/f5f0886f-9115-42d1-ab59-d872f7456d0a/1a08506a-2031-484a-9e68-4d9fd285edb8"
           (reference "#PWR099") (unit 1)
+        )
+      )
+    )
+  )
+  (symbol (lib_id "Connector:TestPoint_Small") (at 149.86 181.61 0) (unit 1)
+    (in_bom yes) (on_board yes) (dnp no)
+    (property "Reference" "TP1" (at 152.146 180.975 0)
+      (effects (font (size 1.27 1.27)) (justify left))
+    )
+    (property "Value" "NRF_TestPoint_IRQ" (at 152.146 183.515 0)
+      (effects (font (size 1.27 1.27)) (justify left))
+    )
+    (property "Footprint" "TestPoint:TestPoint_Pad_D1.0mm" (at 154.94 181.61 0)
+      (effects (font (size 1.27 1.27)) hide)
+    )
+    (property "Datasheet" "~" (at 154.94 181.61 0)
+      (effects (font (size 1.27 1.27)) hide)
+    )
+    (pin "1")
+    (instances
+      (project "Controller_board"
+        (path "/79650e32-6fba-4eaa-902b-d1154ea8c394"
+          (reference "TP1") (unit 1)
+        )
+        (path "/79650e32-6fba-4eaa-902b-d1154ea8c394/7d15cb0c-3f4d-419a-9225-6f102e9a9922"
+          (reference "TP7") (unit 1)
         )
       )
@@
       (effects (font (size 1.27 1.27)) (justify left))
     )
-    (property "Footprint" "Capacitor_SMD:C_0402_1005Metric" (at 169.672 56.261 0)
+    (property "Footprint" "Capacitor_SMD:C_0603_1608Metric" (at 169.672 56.261 0)
       (effects (font (size 1.27 1.27)) hide)
     )
@@
       (effects (font (size 1.27 1.27)))
     )
-    (property "Footprint" "digikey-footprints:RF_SMA_BoardEdge_142-0701-801" (at 140.1826 35.7378 0)
+    (property "Footprint" "Connector_Coaxial:SMA_Molex_73251-2120_EdgeMount_Horizontal" (at 140.1826 35.7378 0)
       (effects (font (size 1.524 1.524)) (justify left) hide)
     )
@@
       (effects (font (size 1.27 1.27)))
     )
-    (property "Footprint" "Inductor_SMD:L_0402_1005Metric" (at 119.7356 48.3108 0)
+    (property "Footprint" "Inductor_SMD:L_0603_1608Metric" (at 119.7356 48.3108 0)
       (effects (font (size 1.27 1.27)) hide)
     )
@@
     )
   )
+  (symbol (lib_id "Connector:TestPoint_Small") (at 149.86 175.768 0) (unit 1)
+    (in_bom yes) (on_board yes) (dnp no)
+    (property "Reference" "TP1" (at 152.146 175.133 0)
+      (effects (font (size 1.27 1.27)) (justify left))
+    )
+    (property "Value" "NRF_TestPoint_CE" (at 152.146 177.673 0)
+      (effects (font (size 1.27 1.27)) (justify left))
+    )
+    (property "Footprint" "TestPoint:TestPoint_Pad_D1.0mm" (at 154.94 175.768 0)
+      (effects (font (size 1.27 1.27)) hide)
+    )
+    (property "Datasheet" "~" (at 154.94 175.768 0)
+      (effects (font (size 1.27 1.27)) hide)
+    )
+    (pin "1")
+    (instances
+      (project "Controller_board"
+        (path "/79650e32-6fba-4eaa-902b-d1154ea8c394"
+          (reference "TP1") (unit 1)
+        )
+        (path "/79650e32-6fba-4eaa-902b-d1154ea8c394/7d15cb0c-3f4d-419a-9225-6f102e9a9922"
+          (reference "TP6") (unit 1)
+        )
+      )
+    )
+  )
   (symbol (lib_id "power:GND") (at 214.503 121.793 0) (unit 1)
     (in_bom yes) (on_board yes) (dnp no) (fields_autoplaced)
@@
       (effects (font (size 1.27 1.27)) (justify left))
     )
-    (property "Footprint" "Inductor_SMD:L_0402_1005Metric" (at 111.0996 44.3738 0)
+    (property "Footprint" "Inductor_SMD:L_0603_1608Metric" (at 111.0996 44.3738 0)
       (effects (font (size 1.27 1.27)) hide)
     )
@@
       (effects (font (size 1.27 1.27)) (justify left))
     )
-    (property "Footprint" "Capacitor_SMD:C_0402_1005Metric" (at 135.9916 44.3738 0)
+    (property "Footprint" "Capacitor_SMD:C_0603_1608Metric" (at 135.9916 44.3738 0)
       (effects (font (size 1.27 1.27)) hide)
     )
@@
       (effects (font (size 1.27 1.27)) (justify left))
     )
-    (property "Footprint" "Capacitor_SMD:C_0402_1005Metric" (at 262.0264 66.2178 0)
+    (property "Footprint" "Capacitor_SMD:C_0603_1608Metric" (at 262.0264 66.2178 0)
       (effects (font (size 1.27 1.27)) hide)
     )
@@
       (effects (font (size 1.27 1.27)) (justify left))
     )
-    (property "Footprint" "Capacitor_SMD:C_0402_1005Metric" (at 130.1496 40.8178 0)
+    (property "Footprint" "Capacitor_SMD:C_0603_1608Metric" (at 130.1496 40.8178 0)
       (effects (font (size 1.27 1.27)) hide)
     )
@@
       (effects (font (size 1.27 1.27)))
     )
-    (property "Footprint" "Inductor_SMD:L_0402_1005Metric" (at 119.7356 40.8178 0)
+    (property "Footprint" "Inductor_SMD:L_0603_1608Metric" (at 119.7356 40.8178 0)
       (effects (font (size 1.27 1.27)) hide)
     )
@@
       (effects (font (size 1.27 1.27)) (justify left))
     )
-    (property "Footprint" "Capacitor_SMD:C_0402_1005Metric" (at 178.562 56.261 0)
-      (effects (font (size 1.27 1.27)) hide)
-    )
+    (property "Footprint" "Capacitor_SMD:C_0603_1608Metric" (at 178.562 56.261 0)
+      (effects (font (size 1.27 1.27)) hide)
+    )
